File: H7_control_board/vibrometer_h7/audio_output.kicad_sch (KiCad schematic)
At the start: 33 parts, among them J901 PH-313D, U901 RC4580, U902 TPA6111A2

Commit message: working through drc errors
Changed lines of the file:
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@@
 	)
 	(symbol
+		(lib_name "RC4580_2")
 		(lib_id "Amplifier_Operational:RC4580")
 		(at 83.82 83.82 0)
@@
 		)
 		(pin "1"
+		)
+		(pin "9"
 		)
 		(instances
@@
 		(dnp no)
 		(property "Reference" "U901"
-			(at 46.482 26.924 0)
-			(effects
-				(font
-					(size 1.27 1.27)
-				)
-				(justify left)
+			(at 51.435 25.146 0)
+			(effects
+				(font
+					(size 1.27 1.27)
+				)
 			)
 		)
 		(property "Value" "RC4580"
-			(at 46.228 38.354 0)
-			(effects
-				(font
-					(size 1.27 1.27)
-				)
-				(justify left)
+			(at 52.197 27.432 0)
+			(effects
+				(font
+					(size 1.27 1.27)
+				)
 			)
 		)
@@
 		(pin "1"
 		)
+		(pin "9"
+		)
 		(instances
 			(project ""
@@
 	)
 	(symbol
+		(lib_name "RC4580_1")
 		(lib_id "Amplifier_Operational:RC4580")
 		(at 82.55 140.97 0)
@@
 		(dnp no)
 		(property "Reference" "U901"
-			(at 86.741 134.366 0)
+			(at 85.725 134.366 0)
 			(effects
 				(font
@@
 		)
 		(property "Value" "RC4580"
-			(at 87.249 136.906 0)
+			(at 86.487 136.652 0)
 			(effects
 				(font
@@
 		(pin "1"
 		)
-		(instances
+		(pin "9"
+		)
+		(instances

Commit message: nearly done....
Parts:
- C901, C904: footprint Capacitor_SMD:C_0402_1005Metric_Pad0.74x0.62mm_HandSolder -> Capacitor_SMD:C_0402_1005Metric
- C906, C907, C908, C911, C913, C914: LCSC C15850 -> C45783
- U902: footprint Package_SO:HVSSOP-8-1EP_3x3mm_P0.65mm_EP1.57x1.89mm -> Package_SO:SOIC-8-1EP_3.9x4.9mm_P1.27mm_EP2.29x3mm
Connections:
- net GND: now also U901.9
Changed lines of the file:
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@@
 	)
 	(junction
+		(at 45.72 43.18)
+		(diameter 0)
+		(color 0 0 0 0)
+	)
+	(junction
 		(at 177.8 95.25)
 		(diameter 0)
@@
 	(wire
 		(pts
+			(xy 45.72 43.18) (xy 45.72 44.45)
+		)
+		(stroke
+			(width 0)
+			(type default)
+		)
+	)
+	(wire
+		(pts
 			(xy 219.71 96.52) (xy 219.71 81.28)
 		)
@@
 	(wire
 		(pts
+			(xy 48.26 39.37) (xy 48.26 43.18)
+		)
+		(stroke
+			(width 0)
+			(type default)
+		)
+	)
+	(wire
+		(pts
 			(xy 172.72 81.28) (xy 172.72 106.68)
 		)
@@
 	(wire
 		(pts
+			(xy 48.26 43.18) (xy 45.72 43.18)
+		)
+		(stroke
+			(width 0)
+			(type default)
+		)
+	)
+	(wire
+		(pts
 			(xy 203.2 128.27) (xy 203.2 129.54)
 		)
@@
 	(wire
 		(pts
-			(xy 45.72 41.91) (xy 45.72 44.45)
+			(xy 45.72 41.91) (xy 45.72 43.18)
 		)
 		(stroke
@@
 			)
 		)
-		(property "Footprint" "Capacitor_SMD:C_0402_1005Metric_Pad0.74x0.62mm_HandSolder"
+		(property "Footprint" "Capacitor_SMD:C_0402_1005Metric"
 			(at 39.37 27.94 0)
 			(effects
@@
 			)
 		)
-		(property "Datasheet" "CL21A106KAYNNNE_C15850.pdf"
+		(property "Datasheet" "https://wmsc.lcsc.com/wmsc/upload/file/pdf/v2/lcsc/2304140030_Samsung-Electro-Mechanics-CL21A226MAQNNNE_C45783.pdf"
 			(at 228.6 104.14 0)
 			(effects
@@
 			)
 		)
-		(property "LCSC" "C15850"
+		(property "LCSC" "C45783"
 			(at 228.6 104.14 0)
 			(effects
@@
 			)
 		)
-		(property "Datasheet" "CL21A106KAYNNNE_C15850.pdf"
+		(property "Datasheet" "https://wmsc.lcsc.com/wmsc/upload/file/pdf/v2/lcsc/2304140030_Samsung-Electro-Mechanics-CL21A226MAQNNNE_C45783.pdf"
 			(at 228.6 96.52 0)
 			(effects
@@
 			)
 		)
-		(property "LCSC" "C15850"
+		(property "LCSC" "C45783"
 			(at 228.6 96.52 0)
 			(effects
@@
 			)
 		)
-		(property "Datasheet" "CL21A106KAYNNNE_C15850.pdf"
+		(property "Datasheet" "https://wmsc.lcsc.com/wmsc/upload/file/pdf/v2/lcsc/2304140030_Samsung-Electro-Mechanics-CL21A226MAQNNNE_C45783.pdf"
 			(at 228.6 115.57 0)
 			(effects
@@
 			)
 		)
-		(property "LCSC" "C15850"
+		(property "LCSC" "C45783"
 			(at 228.6 115.57 0)
 			(effects
@@
 			)
 		)
-		(property "Datasheet" "CL21A106KAYNNNE_C15850.pdf"
+		(property "Datasheet" "https://wmsc.lcsc.com/wmsc/upload/file/pdf/v2/lcsc/2304140030_Samsung-Electro-Mechanics-CL21A226MAQNNNE_C45783.pdf"
 			(at 228.6 119.38 0)
 			(effects
@@
 			)
 		)
-		(property "LCSC" "C15850"
+		(property "LCSC" "C45783"
 			(at 228.6 119.38 0)
 			(effects
@@
 			)
 		)
-		(property "Datasheet" "CL21A106KAYNNNE_C15850.pdf"
+		(property "Datasheet" "https://wmsc.lcsc.com/wmsc/upload/file/pdf/v2/lcsc/2304140030_Samsung-Electro-Mechanics-CL21A226MAQNNNE_C45783.pdf"
 			(at 228.6 100.33 0)
 			(effects
@@
 			)
 		)
-		(property "LCSC" "C15850"
+		(property "LCSC" "C45783"
 			(at 228.6 100.33 0)
 			(effects
@@
 			)
 		)
-		(property "Footprint" "Capacitor_SMD:C_0402_1005Metric_Pad0.74x0.62mm_HandSolder"
+		(property "Footprint" "Capacitor_SMD:C_0402_1005Metric"
 			(at 186.69 95.25 0)
 			(effects
@@
 			)
 		)
-		(property "Datasheet" "CL21A106KAYNNNE_C15850.pdf"
+		(property "Datasheet" "https://wmsc.lcsc.com/wmsc/upload/file/pdf/v2/lcsc/2304140030_Samsung-Electro-Mechanics-CL21A226MAQNNNE_C45783.pdf"
 			(at 228.6 123.19 0)
 			(effects
@@
 			)
 		)
-		(property "LCSC" "C15850"
+		(property "LCSC" "C45783"
 			(at 228.6 123.19 0)
 			(effects
@@
 			)
 		)
-		(property "Footprint" "Package_SO:HVSSOP-8-1EP_3x3mm_P0.65mm_EP1.57x1.89mm"
+		(property "Footprint" "Package_SO:SOIC-8-1EP_3.9x4.9mm_P1.27mm_EP2.29x3mm"
 			(at 193.04 83.058 0)
 			(effects

Commit message: finished analog filter, made a logo :)
Parts:
- C902: value C_Small -> 100n; footprint Capacitor_SMD:C_0603_1608Metric -> Capacitor_SMD:C_0402_1005Metric; LCSC (none) -> C307331
- C905, C912, C916: value C_Small -> 100n
- JP901: value AMP2 FILT BYPASS -> FILT2 BYPASS
- JP902: value AMP1 FILT BYPASS -> FILT1 BYPASS
- R901, R902, R908, R909: value R_Small_US -> 80; footprint Resistor_SMD:R_0402_1005Metric -> Resistor_SMD:R_0603_1608Metric; LCSC (none) -> C3016237
- R904, R911: value R_Small_US -> 5k9; footprint Resistor_SMD:R_0402_1005Metric -> Resistor_SMD:R_0603_1608Metric; LCSC (none) -> C23071
- R905, R912: value R_Small_US -> 10k; LCSC (none) -> C25744
Connections:
- net FILT1_OUT: now reaches C902.1, JP902.1 (A), R904.2, U901.1
- net FILT2_OUT: now reaches C912.1, JP901.1 (A), R911.2, U901.7
Other:
- note added: "C1"
- note added: "C2"
- note added: "R1"
- note added: "R2"
- note added: "R_a"
- note added: "R_b"
- note added: "Voltage gain: A = 1 + R_a / R_b Cutoff freq: f_c = 1/(2Pi*R*C) # assumes R1 = R2, C1 = C2 Quality factor: A = 3 - 1/Q # butterworth filter, Q = 1/sqrt(2)"
- note added: "f_c = 20kHz assume R = 100, C = 1/(2Pi*100*20k) = 79.6e-9 = 80nF # very close to 100nF which is used all over assume C = 100n, R = 1/(2Pi*100n*20k) = 79.6 Ohm Set Q = 1/sqrt(2) = 0.7071 A = 3-1/0.7071 = 1.586 A = 1 + R_a / R_b = 1.586 R_a = 0.586 * R_b assume R_b = 10k, R_a = 5.86k"
- note added: "https://www.electronics-tutorials.ws/filter/second-order-filters.html"
- note removed: "add sallen-key filter with a discrete opamp between DAC output and headphone amp input put solder bridge to bypass the salen-key as a fun little science project"
- moved on the sheet: C905, C916, JP901, JP902, R911, R912, U901B
