File: H7_control_board/vibrometer_h7/SPI_ACCEL.kicad_sch (KiCad schematic)
At the start: 8 parts, among them J601 Conn_01x08_Socket, J602 Conn_01x08_Socket

Commit message: boards sent to JLCPCB!
Connections:
- net ACCEL_MISO: now also J601.6 (Pin_6); no longer J601.5 (Pin_5)
- net ACCEL_MOSI: now also J601.5 (Pin_5); no longer J601.6 (Pin_6)
Changed lines of the file:
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@@
 	(hierarchical_label "ACCEL_MOSI"
 		(shape input)
-		(at 80.01 82.55 180)
+		(at 80.01 85.09 180)
 		(fields_autoplaced yes)
 		(effects
@@
 	(hierarchical_label "ACCEL_MISO"
 		(shape input)
-		(at 80.01 85.09 180)
+		(at 80.01 82.55 180)
 		(fields_autoplaced yes)
 		(effects
