File: H7_control_board/vibrometer_h7/user_interface.kicad_sch (KiCad schematic)
At the start: 13 parts, among them J501 debug_conn, SW501 SW_Push, SW502 SW_Push

Commit message: checked all footprints, made tiny daughterboard
Parts:
- SW501, SW502: LCSC C3010224 -> C221872
Changed lines of the file:
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@@
 			)
 		)
-		(property "Datasheet" "https://www.lcsc.com/datasheet/lcsc_datasheet_2205051716_XKB-Connection-TS-1102SD-A-D-R_C3010224.pdf"
+		(property "Datasheet" "https://www.lcsc.com/datasheet/lcsc_datasheet_2304140030_C-K-PTS645SK50SMTR92LFS_C221872.pdf"
 			(at 124.46 102.87 0)
 			(effects
@@
 			)
 		)
-		(property "LCSC" "C3010224"
+		(property "LCSC" "C221872"
 			(at 124.46 107.95 0)
 			(effects
@@
 			)
 		)
-		(property "Datasheet" "https://www.lcsc.com/datasheet/lcsc_datasheet_2205051716_XKB-Connection-TS-1102SD-A-D-R_C3010224.pdf"
+		(property "Datasheet" "https://www.lcsc.com/datasheet/lcsc_datasheet_2304140030_C-K-PTS645SK50SMTR92LFS_C221872.pdf"
 			(at 123.19 69.85 0)
 			(effects
@@
 			)
 		)
-		(property "LCSC" "C3010224"
+		(property "LCSC" "C221872"
 			(at 123.19 74.93 0)
 			(effects
