File: Hardware/vibecheck_mainboard/USB.kicad_sch (KiCad schematic)
At the start: 29 parts, among them J301 USB_C_Receptacle_USB2.0_16P, U301 USBLC6-2SC6, U302 MT9700, U303 AMS1117-3V3

Commit message: VibeCheck mainboard V1.1 sent to JLCPCB
Changes made to main board:
- audio filter/amplifier gain changed from 1.5 to 1. Changed values of R_in and R_f resistors.
- changed sensor labels on board from 'accel 1' ... to 'sensor 0' ... to match firmware
- updated BOM and DNP parts to make sure they matched better reducing warnings in JLCPCB parts selection process
Parts:
- L302: LCSC C86092 -> C86092
- TP11, TP12, TP302, TP303, TP304, TP305: now left out of the parts list
Changed lines of the file:
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@@
 		(unit 1)
 		(exclude_from_sim no)
-		(in_bom yes)
+		(in_bom no)
 		(on_board no)
 		(dnp yes)
@@
 		(unit 1)
 		(exclude_from_sim no)
-		(in_bom yes)
+		(in_bom no)
 		(on_board yes)
 		(dnp no)
@@
 		(unit 1)
 		(exclude_from_sim no)
-		(in_bom yes)
+		(in_bom no)
 		(on_board yes)
 		(dnp no)
@@
 		(unit 1)
 		(exclude_from_sim no)
-		(in_bom yes)
+		(in_bom no)
 		(on_board yes)
 		(dnp no)
@@
 		(unit 1)
 		(exclude_from_sim no)
-		(in_bom yes)
+		(in_bom no)
 		(on_board yes)
 		(dnp no)
@@
 			)
 		)
-		(property "LCSC" "C86092 "
+		(property "LCSC" "C86092"
 			(at 222.25 60.96 0)
 			(effects
@@
 		(unit 1)
 		(exclude_from_sim no)
-		(in_bom yes)
-		(on_board yes)
-		(dnp no)
+		(in_bom no)
+		(on_board yes)
+		(dnp no)
