File: Hardware/vibecheck_mainboard/led_strobe.kicad_sch (KiCad schematic)
At the start: 49 parts, among them Q1001 NTR4170N, Q1002 NTR4170N, Q1003 NTR4170N

Commit message: VibeCheck mainboard V1.1 sent to JLCPCB
Changes made to main board:
- audio filter/amplifier gain changed from 1.5 to 1. Changed values of R_in and R_f resistors.
- changed sensor labels on board from 'accel 1' ... to 'sensor 0' ... to match firmware
- updated BOM and DNP parts to make sure they matched better reducing warnings in JLCPCB parts selection process
Parts:
- C1001, TP1001, TP1002, TP1003: now left out of the parts list
- D1001, D1002, D1003, D1004, D1005, D1006, D1007, D1008, D1009, D1010, D1011, D1012: LCSC C540978 -> C540978
- R1001, R1002, R1003, R1004, R1005, R1006, R1007, R1008, R1009, R1010, R1011, R1012: LCSC C5552472 -> C17622
Changed lines of the file:
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@@
 		(unit 1)
 		(exclude_from_sim no)
-		(in_bom yes)
+		(in_bom no)
 		(on_board yes)
 		(dnp no)
@@
 			)
 		)
-		(property "LCSC" "C540978 "
+		(property "LCSC" "C540978"
 			(at 161.29 73.66 0)
 			(effects
@@
 			)
 		)
-		(property "LCSC" "C5552472 "
+		(property "LCSC" "C17622"
 			(at 237.49 63.5 0)
 			(effects
@@
 			)
 		)
-		(property "LCSC" "C5552472 "
+		(property "LCSC" "C17622"
 			(at 110.49 63.5 0)
 			(effects
@@
 			)
 		)
-		(property "LCSC" "C540978 "
+		(property "LCSC" "C540978"
 			(at 212.09 73.66 0)
 			(effects
@@
 			)
 		)
-		(property "LCSC" "C540978 "
+		(property "LCSC" "C540978"
 			(at 224.79 73.66 0)
 			(effects
@@
 			)
 		)
-		(property "LCSC" "C5552472 "
+		(property "LCSC" "C17622"
 			(at 212.09 63.5 0)
 			(effects
@@
 			)
 		)
-		(property "LCSC" "C5552472 "
+		(property "LCSC" "C17622"
 			(at 186.69 63.5 0)
 			(effects
@@
 			)
 		)
-		(property "LCSC" "C5552472 "
+		(property "LCSC" "C17622"
 			(at 123.19 63.5 0)
 			(effects
@@
 			)
 		)
-		(property "LCSC" "C5552472 "
+		(property "LCSC" "C17622"
 			(at 148.59 63.5 0)
 			(effects
@@
 			)
 		)
-		(property "LCSC" "C540978 "
+		(property "LCSC" "C540978"
 			(at 237.49 73.66 0)
 			(effects
@@
 			)
 		)
-		(property "LCSC" "C540978 "
+		(property "LCSC" "C540978"
 			(at 199.39 73.66 0)
 			(effects
@@
 			)
 		)
-		(property "LCSC" "C5552472 "
+		(property "LCSC" "C17622"
 			(at 135.89 63.5 0)
 			(effects
@@
 			)
 		)
-		(property "LCSC" "C540978 "
+		(property "LCSC" "C540978"
 			(at 123.19 73.66 0)
 			(effects
@@
 			)
 		)
-		(property "LCSC" "C5552472 "
+		(property "LCSC" "C17622"
 			(at 97.79 63.5 0)
 			(effects
@@
 			)
 		)
-		(property "LCSC" "C5552472 "
+		(property "LCSC" "C17622"
 			(at 224.79 63.5 0)
 			(effects
@@
 			)
 		)
-		(property "LCSC" "C5552472 "
+		(property "LCSC" "C17622"
 			(at 173.99 63.5 0)
 			(effects
@@
 		(unit 1)
 		(exclude_from_sim no)
-		(in_bom yes)
+		(in_bom no)
 		(on_board yes)
 		(dnp no)
@@
 			)
 		)
-		(property "LCSC" "C540978 "
+		(property "LCSC" "C540978"
 			(at 186.69 73.66 0)
 			(effects
@@
 			)
 		)
-		(property "LCSC" "C540978 "
+		(property "LCSC" "C540978"
 			(at 110.49 73.66 0)
 			(effects
@@
 			)
 		)
-		(property "LCSC" "C5552472 "
+		(property "LCSC" "C17622"
 			(at 199.39 63.5 0)
 			(effects
@@
 			)
 		)
-		(property "LCSC" "C540978 "
+		(property "LCSC" "C540978"
 			(at 173.99 73.66 0)
 			(effects
@@
 			)
 		)
-		(property "LCSC" "C540978 "
+		(property "LCSC" "C540978"
 			(at 148.59 73.66 0)
 			(effects
@@
 			)
 		)
-		(property "LCSC" "C540978 "
+		(property "LCSC" "C540978"
 			(at 97.79 73.66 0)
 			(effects
@@
 		(unit 1)
 		(exclude_from_sim no)
-		(in_bom yes)
+		(in_bom no)
 		(on_board yes)
 		(dnp yes)
@@
 			)
 		)
-		(property "LCSC" "C5552472 "
+		(property "LCSC" "C17622"
 			(at 161.29 63.5 0)
 			(effects
@@
 		(unit 1)
 		(exclude_from_sim no)
-		(in_bom yes)
+		(in_bom no)
 		(on_board yes)
 		(dnp no)
@@
 			)
 		)
-		(property "LCSC" "C540978 "
+		(property "LCSC" "C540978"
 			(at 135.89 73.66 0)
 			(effects
