File: Hardware/vibecheck_mainboard/user_interface.kicad_sch (KiCad schematic)
At the start: 13 parts, among them J501 debug_conn, SW501 SW_Push, SW502 SW_Push

Commit message: VibeCheck mainboard V1.1 sent to JLCPCB
Changes made to main board:
- audio filter/amplifier gain changed from 1.5 to 1. Changed values of R_in and R_f resistors.
- changed sensor labels on board from 'accel 1' ... to 'sensor 0' ... to match firmware
- updated BOM and DNP parts to make sure they matched better reducing warnings in JLCPCB parts selection process
Parts:
- J501: now left out of the parts list
Changed lines of the file:
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@@
 		(unit 1)
 		(exclude_from_sim no)
-		(in_bom yes)
+		(in_bom no)
 		(on_board yes)
 		(dnp yes)
